Commit message: change files

File: src/holybro_model/urdf/model_lidar.urdf (robot description, URDF)
Before this commit: robot holybro, 21 links, 20 joints
Joints:
- joint livox_frame_joint: origin xyz=0.0 0.0 0.0 rpy=0.0 0.0 3.1415926 -> xyz=0.0 0.0 0.0 rpy=0.0 0.0 0.0

Commit message: commit

File: src/holybro_model/urdf/model_lidar.urdf (robot description, URDF)
Before this commit: robot holybro, 21 links, 20 joints
Joints:
- joint livox_frame_joint: origin xyz=0.0 0.0 0.0 rpy=0.0 0.0 0.0 -> xyz=0.0 0.0 0.0 rpy=0 0 0
